Commit message: Repository cleanup

File: Antonio_Docker/antonio_ws/src/antonio_description/src/description/antonio_description.urdf (robot description, URDF)
Before this commit: robot antonio, 7 links, 6 joints
Links:
- removed link camera_depth_frame
- added link Floor_scan, mass 0.125; collision cylinder length=0.055 radius=0.0508; visual cylinder length=0.055 radius=0.0508
- added link wheels_center; visual sphere radius=0.01
- link imu_link: geometry collision box size=0.1 0.1 0.1; visual box size=0.01 0.01 0.01
Joints:
- removed joint camera_depth_joint
- added joint Floor_scan_joint: type fixed, parent base_link, child Floor_scan, origin xyz=0.17 0 0.135 rpy=0 0.785398163 0
- added joint wheels_center_joint: type fixed, parent base_link, child wheels_center, origin xyz=-0.13 0.0 0 rpy=0 0 0
- joint camera_joint: origin xyz=0.215 0 0.05 rpy=0 0 0 -> xyz=0 0 0.86 rpy=0 0.77 0
- joint imu_joint: origin xyz=0 0 0.01 -> xyz=0 0 0.09 rpy=0 0 0
- joint lidar_joint: origin xyz=0 0 0.12 rpy=0 0 0 -> xyz=0.0 0 0.19 rpy=0 0 3.141592

Commit message: Minor changes

File: Antonio_Docker/antonio_ws/src/antonio_description/src/description/antonio_description.urdf (robot description, URDF)
Before this commit: robot antonio, 8 links, 7 joints
Joints:
- joint Floor_scan_joint: origin xyz=0.17 0 0.135 rpy=0 0.785398163 0 -> xyz=0.17 0 0.135 rpy=0 0.5934 0

Commit message: add pcd_manag_pkg

File: Antonio_Docker/antonio_ws/src/antonio_description/src/description/antonio_description.urdf (robot description, URDF)
Before this commit: robot antonio, 8 links, 7 joints
Joints:
- joint wheels_center_joint: child wheels_center -> base_link; origin xyz=-0.13 0.0 0 rpy=0 0 0 -> xyz=-0.11 0.0 0 rpy=0 0 0; parent base_link -> wheels_center
